File: KiCad files/Sheet2.kicad_sch (KiCad schematic)
At the start: 56 parts, among them J10 Conn_01x11_Female, J11 Conn_01x11_Male, J12 Conn_01x11_Male, J3 Screw_Terminal_01x02, J4 Screw_Terminal_01x02, J5 Conn_01x04_Female, J6 OLED, J7 Conn_01x05_Female, J8 Conn_01x05_Male, J9 Conn_01x11_Female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

Commit message: Update
Parts:
- removed BZ1: Buzzer, ESP32IoTPlatform:PS1240P02BT, symbol Device:Buzzer
- removed C19: 100n/50V, Capacitor_SMD:C_0805_2012Metric, symbol Device:C_Small
- removed C20: 10u/16V, Capacitor_SMD:C_0805_2012Metric, symbol Device:C_Small
- removed D12: S1BB-13-F, Diode_SMD:D_SMA, symbol Device:D_Small
- removed D13: Green, LED_SMD:LED_0805_2012Metric, symbol Device:LED_Small
- removed H1, H2, H3, H4: MountingHole, MountingHole:MountingHole_3.2mm_M3_Pad_Via, symbol Mechanical:MountingHole
- removed J10, J9: Conn_01x11_Female, Connector_PinSocket_2.54mm:PinSocket_1x11_P2.54mm_Vertical, symbol Connector:Conn_01x11_Female
- removed J11, J12: Conn_01x11_Male, Connector_PinHeader_2.54mm:PinHeader_1x11_P2.54mm_Vertical, symbol Connector:Conn_01x11_Male
- removed J3, J4: Screw_Terminal_01x02, TerminalBlock_Phoenix:TerminalBlock_Phoenix_MKDS-1,5-2-5.08_1x02_P5.08mm_Horizontal, symbol Connector:Screw_Terminal_01x02
- removed J5: Conn_01x04_Female, ESP32IoTPlatform:PinSocket_1x04_P2.54mm_Vertical, symbol Connector:Conn_01x04_Female
- removed J6: OLED, ESP32IoTPlatform:OLED, symbol Connector:Conn_01x04_Female
- removed J7: Conn_01x05_Female, Connector_PinSocket_2.54mm:PinSocket_1x05_P2.54mm_Vertical, symbol Connector:Conn_01x05_Female
- removed J8: Conn_01x05_Male, Connector_PinHeader_2.54mm:PinHeader_1x05_P2.54mm_Vertical, symbol Connector:Conn_01x05_Male
- removed Q3: IRLZ44N, Package_TO_SOT_THT:TO-220-3_Vertical, symbol Transistor_FET:IRLZ44N
- removed Q4, Q5: SI2302DS, Package_TO_SOT_SMD:SOT-23, symbol Transistor_FET:IRLZ44N
- removed Q6: Q_DUAL_NPN_UMH3N, Package_TO_SOT_SMD:SOT-363_SC-70-6, symbol Device:Q_DUAL_NPN_NPN_BRT_E1B1C2E2B2C1
- removed Q7: Q_DUAL_PNP_BCM857BS, Package_TO_SOT_SMD:SOT-363_SC-70-6, symbol Device:Q_DUAL_PNP_PNP_BRT_E1B1C2E2B2C1
- removed Q8: CJ2301, Package_TO_SOT_SMD:SOT-23, symbol Transistor_FET:Si2319CDS
- removed R14, R17, R20, R27, R29: 10k, Resistor_SMD:R_0805_2012Metric, symbol Device:R_Small
- removed R15: 1k, Resistor_SMD:R_0805_2012Metric, symbol Device:R_Small
- removed R16: 1k5, Resistor_SMD:R_0805_2012Metric, symbol Device:R_Small
- removed R18: 470R, Resistor_SMD:R_0805_2012Metric, symbol Device:R_Small
- removed R19: LDR, OptoDevice:R_LDR_10x8.5mm_P7.6mm_Vertical, symbol Sensor_Optical:LDR03
- removed R21: 243R, Resistor_SMD:R_0805_2012Metric, symbol Device:R_Small
- removed R22, R23, R24, R25, R26: 2k, Resistor_SMD:R_0805_2012Metric, symbol Device:R_Small
- removed R28: 47k, Resistor_SMD:R_0805_2012Metric, symbol Device:R_Small
- removed RV1: 10k, ESP32IoTPlatform:Potentiometer_Bourns_3386P_Vertical, symbol Device:R_POT_Small
- removed SD1: microSD-MOLEX-473521001, ESP32IoTPlatform:MOLEX_47352-1001, symbol ESP32IoTPlatform_simboli:microSD-MOLEX-473521001
- removed SW10, SW9: SW_x02, Button_Switch_SMD:SW_DIP_SPSTx02_Slide_6.7x6.64mm_W6.73mm_P2.54mm_LowProfile_JPin, symbol Switch:SW_DIP_x02
- removed SW11: SW_x03, Button_Switch_SMD:SW_DIP_SPSTx03_Slide_6.7x9.18mm_W6.73mm_P2.54mm_LowProfile_JPin, symbol Switch:SW_DIP_x03
- removed SW14, SW15, SW16, SW18, SW8: SW_x01, Button_Switch_SMD:SW_DIP_SPSTx01_Slide_6.7x4.1mm_W6.73mm_P2.54mm_LowProfile_JPin, symbol Switch:SW_DIP_x01
- removed SW17: SW_x05, Button_Switch_SMD:SW_DIP_SPSTx05_Slide_6.7x14.26mm_W6.73mm_P2.54mm_LowProfile_JPin, symbol Switch:SW_DIP_x05
- removed SW19: SW_x04, Button_Switch_SMD:SW_DIP_SPSTx04_Slide_6.7x11.72mm_W6.73mm_P2.54mm_LowProfile_JPin, symbol Switch:SW_DIP_x04
- removed T1: SKRHABE010, ESP32IoTPlatform:Alps_SKRHABE010, symbol ESP32IoTPlatform_simboli:SKRHABE010
- removed TP1: Touchpad, ESP32IoTPlatform:Touchpad, symbol ESP32IoTPlatform_simboli:Touchpad
- removed U7: L80-M39, ESP32IoTPlatform:L80-M39, symbol ESP32IoTPlatform_simboli:L80-M39
Connections:
- no-connect marks 3 -> 0
Other:
- note removed: "AUTO-PROGRAM"
- note removed: "FOTOOTPORNIK"
- note removed: "GPS"
- note removed: "HC-SR04"
- note removed: "HEADERI"
- note removed: "JOYSTICK"
- note removed: "MOSFET"
- note removed: "NAPAJANJE 2"
- note removed: "OLED"
- note removed: "POTENCIOMETAR"
- note removed: "RUPE"
- note removed: "TOUCHPAD"
- note removed: "ZUJALICA"
- note removed: "microSD"
