File: KiCad files/senzori.kicad_sch (KiCad schematic)
At the start: 28 parts, among them J5 Conn_01x04_Female, Q4 SI2302DS, SW11 SW_x03, SW14 SW_x01, SW15 SW_x01, SW16 SW_x01, SW17 SW_x05, SW9 SW_x02, T1 SKRHABE010, U7 L80-M39

Commit message: update
Parts:
- R19: footprint OptoDevice:R_LDR_10x8.5mm_P7.6mm_Vertical -> OptoDevice:R_LDR_7x6mm_P5.1mm_Vertical
Changed lines of the file:
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@@
       (effects (font (size 1.27 1.27)) (justify left))
     )
-    (property "Footprint" "OptoDevice:R_LDR_10x8.5mm_P7.6mm_Vertical" (id 2) (at 140.97 75.565 90)
+    (property "Footprint" "OptoDevice:R_LDR_7x6mm_P5.1mm_Vertical" (id 2) (at 140.97 75.565 90)
       (effects (font (size 1.27 1.27)) hide)
     )
