File: KiCad files/I2C.kicad_sch (KiCad schematic)
At the start: 16 parts, among them J6 OLED, SW10 SW_x02, SW2 SW_x02, SW3 SW_x02, SW4 SW_x02, U4 BME280, U5 MPU-6050

Commit message: route
Connections:
- net at J6.3 (Pin_3): now also SW10.3; no longer SW10.4
- net at J6.4 (Pin_4): now also SW10.4; no longer SW10.3
Changed lines of the file:
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@@
-    (stroke (width 0) (type default) (color 0 0 0 0))
-  )
-  (wire (pts (xy 81.915 100.33) (xy 81.915 102.87))
-    (stroke (width 0) (type default) (color 0 0 0 0))
-  )
-  (wire (pts (xy 80.645 100.33) (xy 80.645 97.79))
     (stroke (width 0) (type default) (color 0 0 0 0))
   )
@@
   )
   (wire (pts (xy 74.295 85.09) (xy 79.375 85.09))
-    (stroke (width 0) (type default) (color 0 0 0 0))
-  )
-  (wire (pts (xy 83.185 100.33) (xy 81.915 100.33))
     (stroke (width 0) (type default) (color 0 0 0 0))
   )
@@
     (stroke (width 0) (type default) (color 0 0 0 0))
   )
-  (wire (pts (xy 79.375 100.33) (xy 80.645 100.33))
-    (stroke (width 0) (type default) (color 0 0 0 0))
-  )
   (wire (pts (xy 238.125 78.74) (xy 236.855 78.74))
     (stroke (width 0) (type default) (color 0 0 0 0))
@@
     (stroke (width 0) (type default) (color 0 0 0 0))
   )
-  (wire (pts (xy 81.915 102.87) (xy 79.375 102.87))
+  (wire (pts (xy 81.28 97.79) (xy 83.185 97.79))
     (stroke (width 0) (type default) (color 0 0 0 0))
   )
@@
     (stroke (width 0) (type default) (color 0 0 0 0))
   )
-  (wire (pts (xy 80.645 97.79) (xy 83.185 97.79))
-    (stroke (width 0) (type default) (color 0 0 0 0))
-  )
   (wire (pts (xy 236.855 72.39) (xy 234.315 72.39))
     (stroke (width 0) (type default) (color 0 0 0 0))
@@
   )
   (wire (pts (xy 235.585 95.25) (xy 239.395 95.25))
+    (stroke (width 0) (type default) (color 0 0 0 0))
+  )
+  (wire (pts (xy 79.375 100.33) (xy 83.185 100.33))
     (stroke (width 0) (type default) (color 0 0 0 0))
   )
@@
     (stroke (width 0) (type default) (color 0 0 0 0))
   )
+  (wire (pts (xy 81.28 102.87) (xy 81.28 97.79))
+    (stroke (width 0) (type default) (color 0 0 0 0))
+  )
   (wire (pts (xy 53.975 67.31) (xy 53.975 64.77))
     (stroke (width 0) (type default) (color 0 0 0 0))
@@
     (stroke (width 0) (type default) (color 0 0 0 0))
   )
+  (wire (pts (xy 79.375 102.87) (xy 81.28 102.87))
+    (stroke (width 0) (type default) (color 0 0 0 0))
+  )
