File: KiCad files/napajanje.kicad_sch (KiCad schematic)
At the start: 13 parts, among them IC1 ME6211C33M5G, Q1 CJ2301, U3 TP4054

Commit message: route
Parts:
- JST1: footprint Connector_JST:JST_PH_B2B-PH-K_1x02_P2.00mm_Vertical -> ESP32IoTPlatform:A2001WR-S-2P_JST2.0
Changed lines of the file:
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@@
       (effects (font (size 1.27 1.27)) (justify left))
     )
-    (property "Footprint" "Connector_JST:JST_PH_B2B-PH-K_1x02_P2.00mm_Vertical" (id 2) (at 126.365 64.77 0)
+    (property "Footprint" "ESP32IoTPlatform:A2001WR-S-2P_JST2.0" (id 2) (at 126.365 64.77 0)
       (effects (font (size 1.27 1.27)) hide)
     )
