File: KiCad files/ESP32IoTPlatform.kicad_pcb (KiCad board)
At the start: 2 copper layers, 190.8 x 105.2 mm, 124 parts, among them IC1 ME6211C33M5G, J1 USB_B_Micro, J10 Conn_01x11_Female, J11 Conn_01x11_Male, J12 Conn_01x11_Male, J2 Screw_Terminal_01x03, J3 Screw_Terminal_01x02, J4 Screw_Terminal_01x02, J5 Conn_01x04_Female, J6 OLED, J7 Conn_01x05_Female, J8 Conn_01x05_Male, J9 Conn_01x11_Female, K1 SANYOU_SRD_Form_C, Q1 CJ2301, Q2 S8050G, Q3 IRLZ44N, Q4 SI2302DS, Q5 SI2302DS, Q6 Q_DUAL_NPN_UMH3N, Q7 Q_DUAL_PNP_BCM857BS, Q8 CJ2301, SW1 SW_Push, SW10 SW_x02, SW11 SW_x03, SW14 SW_x01, SW15 SW_x01, SW16 SW_x01, SW17 SW_x05, SW18 SW_x01, SW19 SW_x04, SW2 SW_x02, SW3 SW_x02, SW4 SW_x02, SW5 SW_x01, SW6 SW_x01, SW7 SW_x01, SW8 SW_x01, SW9 SW_x02, T1 SKRHABE010, U1 ESP32-WROOM-32D, U2 CP2104, U3 TP4054, U4 BME280, U5 MPU-6050, U6 PC817, U7 L80-M39

Commit message: Update
Parts:
- removed C18: 100n/50V, Capacitor_SMD:C_0805_2012Metric
- removed D8: WS2812B, LED_SMD:LED_WS2812B_PLCC4_5.0x5.0mm_P3.2mm
- added R30: 470, Resistor_SMD:R_0805_2012Metric, F.Cu at (160.2, 56.0)
- added R31: 330, Resistor_SMD:R_0805_2012Metric, F.Cu at (169.0, 56.0)
- added R32: 330, Resistor_SMD:R_0805_2012Metric, F.Cu at (160.2, 62.2)
- C3: value 1000u -> 1500u
- R11: value 80R -> 330
- R18: value 470R -> 470
- R2, R3: value 330R -> 330
- R21, R4: value 243R -> 243
- moved T1 4.41 mm to (104.3, 128.0)
- moved SW16 3.81 mm to (76.6, 118.9)
Connections:
- net Net-(SD1-Pad5) renamed SCK
- D11 pad 1: Net-(D11-Pad1) -> +5V
- D5 pad 4: Net-(D5-Pad4) -> Net-(R30-Pad1)
- D7 pad 2: Net-(D7-Pad2) -> unconnected-(D7-Pad2)
- IC1 pad 4: Net-(IC1-Pad4) -> unconnected-(IC1-Pad4)
- J1 pad 4: Net-(J1-Pad4) -> unconnected-(J1-Pad4)
- J1 pad 6: Net-(J1-Pad6) -> unconnected-(J1-Pad6)
- K1 pad 5: Net-(D11-Pad1) -> +5V
- Q3 pad 1: Net-(Q3-Pad1) -> Net-(R14-Pad1)
- Q4 pad 1: Net-(Q4-Pad1) -> Net-(R17-Pad1)
- R14 pad 1: Net-(Q3-Pad1) -> Net-(R14-Pad1)
- R17 pad 1: Net-(Q4-Pad1) -> Net-(R17-Pad1)
- SD1 pad 1: Net-(SD1-Pad1) -> unconnected-(SD1-Pad1)
- SD1 pad 2: Net-(SD1-Pad2) -> CS
- SD1 pad 3: Net-(SD1-Pad3) -> MOSI
- SD1 pad 7: Net-(SD1-Pad7) -> MISO
- SD1 pad 8: Net-(SD1-Pad8) -> unconnected-(SD1-Pad8)
- SW10 pad 1: IO22 -> IO21
- SW10 pad 2: IO21 -> IO22
- SW17 pad 1: IO2 -> IO23
- SW17 pad 2: IO15 -> IO18
- SW17 pad 3: IO25 -> IO2
- SW17 pad 4: IO23 -> IO15
- SW17 pad 5: IO18 -> IO25
- SW19 pad 1: IO5 -> IO23
- SW19 pad 2: IO23 -> IO19
- SW19 pad 4: IO19 -> IO5
- SW19 pad 5: Net-(SD1-Pad7) -> CS
- SW19 pad 7: Net-(SD1-Pad3) -> MISO
- SW19 pad 8: Net-(SD1-Pad2) -> MOSI
- SW2 pad 1: IO21 -> IO22
- SW2 pad 2: IO22 -> IO21
- SW4 pad 1: IO21 -> IO22
- SW4 pad 2: IO22 -> IO21
- SW5 pad 2: Net-(D5-Pad4) -> Net-(SW5-Pad2)
- SW8 pad 2: Net-(Q3-Pad1) -> Net-(SW8-Pad2)
- T1 pad 7: Net-(T1-Pad7) -> unconnected-(T1-Pad7)
- T1 pad 8: Net-(T1-Pad8) -> unconnected-(T1-Pad8)
- U1 pad 17: Net-(U1-Pad17) -> unconnected-(U1-Pad17)
- U1 pad 18: Net-(U1-Pad18) -> unconnected-(U1-Pad18)
- U1 pad 19: Net-(U1-Pad19) -> unconnected-(U1-Pad19)
- U1 pad 20: Net-(U1-Pad20) -> unconnected-(U1-Pad20)
- U1 pad 21: Net-(U1-Pad21) -> unconnected-(U1-Pad21)
- U1 pad 22: Net-(U1-Pad22) -> unconnected-(U1-Pad22)
- U1 pad 32: Net-(U1-Pad32) -> unconnected-(U1-Pad32)
- U2 pad 1: Net-(U2-Pad1) -> unconnected-(U2-Pad1)
- U2 pad 10: Net-(U2-Pad10) -> unconnected-(U2-Pad10)
- U2 pad 11: Net-(U2-Pad11) -> unconnected-(U2-Pad11)
- U2 pad 12: Net-(U2-Pad12) -> unconnected-(U2-Pad12)
- U2 pad 15: Net-(U2-Pad15) -> unconnected-(U2-Pad15)
- U2 pad 16: Net-(U2-Pad16) -> unconnected-(U2-Pad16)
- U2 pad 17: Net-(U2-Pad17) -> unconnected-(U2-Pad17)
- U2 pad 18: Net-(U2-Pad18) -> unconnected-(U2-Pad18)
- U2 pad 22: Net-(U2-Pad22) -> unconnected-(U2-Pad22)
- U2 pad 24: Net-(U2-Pad24) -> unconnected-(U2-Pad24)
- U2 pad 9: Net-(U2-Pad9) -> unconnected-(U2-Pad9)
- U5 pad 12: Net-(U5-Pad12) -> unconnected-(U5-Pad12)
- U5 pad 6: Net-(U5-Pad6) -> unconnected-(U5-Pad6)
- U5 pad 7: Net-(U5-Pad7) -> unconnected-(U5-Pad7)
- U6 pad 4: Net-(D11-Pad1) -> +5V
- U7 pad 11: Net-(U7-Pad11) -> unconnected-(U7-Pad11)
- U7 pad 6: Net-(Q4-Pad1) -> Net-(U7-Pad6)
- U7 pad 7: Net-(U7-Pad7) -> unconnected-(U7-Pad7)
- U7 pad 8: Net-(U7-Pad8) -> unconnected-(U7-Pad8)
Other:
- net class Default removed
- board text added: "DESNO"
- board text added: "DOLJE"
- board text added: "GORE"
- board text added: "GPS_~{RES}"
- board text added: "LIJEVO"
- board text added: "POTVRDA"
- board text added: "SENZOR DODIRA"
- board text added: "UPRAVLJAČKA RUČICA"
- board text removed: "GPS_~RES~"
- board text removed: "JOY_A"
- board text removed: "JOY_B"
- board text removed: "JOY_C"
- board text removed: "JOY_CEN"
- board text removed: "JOY_D"
- board text removed: "TOUCHPAD"
- board text removed: "TP"

Commit message: update
Parts:
- removed the G*** at (132.6, 89.8)

Commit message: update
Parts:
- moved SD1 158.3 mm to (114.9, 50.6), turned to 180 degrees
- moved G*** 149.0 mm to (4.00, 141.0), turned to 0 degrees
- moved SW19 121.0 mm to (96.1, 49.5), turned to 0 degrees
- moved R31 112.1 mm to (70.1, 108.7), turned to 180 degrees
- moved G*** 57.9 mm to (126.1, 22.6)
- moved Q5 57.9 mm to (125.6, 15.6)
- moved R27 57.9 mm to (125.6, 20.3)
- moved BZ1 57.9 mm to (134.7, 16.9)
- moved SW18 57.9 mm to (120.4, 19.7)
- moved R30 50.2 mm to (123.7, 90.4), turned to 90 degrees
- moved R7 30.4 mm to (70.1, 45.5), turned to 0 degrees
- moved R6 27.2 mm to (70.1, 48.9), turned to 0 degrees
- moved G*** 26.4 mm to (100.7, 109.9)
- moved C8 21.8 mm to (132.3, 72.3)
- moved G*** 21.6 mm to (127.7, 64.7)
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Other:
- board size 190.8 x 105.2 mm -> 190 x 105.2 mm
- board text added: "AKCELEROMETAR"
- board text added: "CS"
- board text added: "MISO"
- board text added: "MOSI"
- board text added: "RGB1"
- board text added: "RGB2"
- board text added: "RGB3"
- board text added: "SCK"
- board text added: "SENZOR TEMPERATURE"
- board text added: "microSD"
- board text removed: "BME280"
- board text removed: "ESP32 IoTPlatfom v3.0"
- board text removed: "Josip Kordek"
- board text removed: "MPU6050"

Commit message: update
Parts:
- R19: footprint OptoDevice:R_LDR_10x8.5mm_P7.6mm_Vertical -> OptoDevice:R_LDR_7x6mm_P5.1mm_Vertical
- moved R21 105.1 mm to (103.4, 86.0)
- moved SW8 100.2 mm to (70.5, 98.9)
- moved SW15 96.7 mm to (106.7, 95.2), turned to 180 degrees
- moved SW7 96.4 mm to (102.6, 137.2), turned to 180 degrees
- moved R20 95.9 mm to (96.6, 114.2)
- moved BZ1 95.8 mm to (230.2, 25.1)
- moved C14 95.8 mm to (261.7, 111.5)
- moved C5 95.8 mm to (266.1, 93.7)
- moved C8 95.8 mm to (227.8, 80.6)
- moved D1 95.8 mm to (269.5, 84.6)
- moved D3 95.8 mm to (251.8, 102.7)
- moved D9 95.8 mm to (141.7, 96.7)
- moved G*** 95.8 mm to (223.2, 73.0)
- moved G*** 95.8 mm to (196.2, 118.2)
- moved G*** 95.8 mm to (221.5, 30.8)
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Other:
- board text added: "+"
- board text added: "-"
- board text removed: "M+"
- board text removed: "M-"

Commit message: logos
Parts:
- added G***: LOGO, ESP32IoTPlatform:kicad_logo, F.Cu at (62.2, 53.4)
- added G***: LOGO, ESP32IoTPlatform:cloud_logo, F.Cu at (226.4, 62.2)
- moved BZ1 184.0 mm to (51.4, 69.0), turned to 0 degrees
- moved Q5 167.0 mm to (60.6, 70.2), turned to -90 degrees
- moved R27 164.7 mm to (60.6, 65.5), turned to 180 degrees
- moved G*** 154.1 mm to (72.2, 69.0)
- moved SW18 149.1 mm to (70.8, 62.6), turned to 180 degrees
- moved SW1 31.4 mm to (99.8, 40.8)
- moved R16 1.14 mm to (54.0, 86.6)
- moved J5 1.14 mm to (50.1, 78.9)
- moved R15 1.14 mm to (54.0, 82.9)
- moved SW9 1.14 mm to (67.6, 83.1)
- moved G*** 0.53 mm to (99.8, 148.8)
Other:
- board text added: "ESP32 IoTPlatform V4.0"

Commit message: route
Parts:
- JST1: footprint Connector_JST:JST_PH_B2B-PH-K_1x02_P2.00mm_Vertical -> ESP32IoTPlatform:A2001WR-S-2P_JST2.0
- moved R32 194.8 mm to (63.0, 99.0), turned to 180 degrees
- moved R29 188.2 mm to (98.3, 79.2)
- moved R28 187.6 mm to (94.5, 79.2)
- moved C4 187.6 mm to (89.0, 55.8), turned to 90 degrees
- moved Q8 185.7 mm to (96.4, 74.6), turned to 90 degrees
- moved Q7 181.7 mm to (109.1, 79.1)
- moved R2 181.6 mm to (88.8, 68.6), turned to -90 degrees
- moved D1 181.0 mm to (88.8, 74.0), turned to -90 degrees
- moved Q6 179.4 mm to (107.4, 69.4)
- moved C5 178.4 mm to (91.8, 55.8), turned to 90 degrees
- moved Q1 176.5 mm to (96.2, 61.2), turned to 90 degrees
- moved U2 175.4 mm to (90.4, 62.2), turned to -90 degrees
- moved R3 171.8 mm to (92.0, 68.6), turned to -90 degrees
- moved D2 170.7 mm to (92.0, 74.0), turned to -90 degrees
- moved R10 167.0 mm to (96.4, 69.4)
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Connections:
- J6 pad 3: Net-(J6-Pad3) -> Net-(SW10-Pad3)
- J6 pad 4: Net-(J6-Pad4) -> Net-(SW10-Pad4)
- SW10 pad 3: Net-(J6-Pad4) -> Net-(SW10-Pad3)
- SW10 pad 4: Net-(J6-Pad3) -> Net-(SW10-Pad4)
Routing:
- net IO22: track 0.00 -> 179.3 mm, vias 0 -> 5
- net IO23: track 0.00 -> 178.1 mm
- net IO21: track 0.00 -> 176.1 mm, vias 0 -> 5
- net IO18: track 0.00 -> 169.3 mm
- net IO33: track 0.00 -> 126.0 mm
- net IO25: track 0.00 -> 122.7 mm, vias 0 -> 2
- net IO19: track 0.00 -> 111.4 mm, vias 0 -> 2
- net IO32: track 0.00 -> 107.3 mm
- net IO15: track 0.00 -> 81.4 mm
- net IO35: track 0.00 -> 81.2 mm
- net IO14: track 0.00 -> 77.4 mm
- net IO2: track 0.00 -> 76.6 mm
- net IO5: track 0.00 -> 73.6 mm
- net IO26: track 0.00 -> 72.6 mm, vias 0 -> 1
- net IO4: track 0.00 -> 68.3 mm
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- added copper zone on F.Cu, net +3V3
- added copper zone on F.Cu, net +BATT
- added copper zone on B.Cu, net GND
- added copper zone on F.Cu, net GND
Other:
- board text added: "CHRG"
- board text added: "RX"
- board text added: "TX"

Commit message: route2
Routing:
- net VBUS: track 0.00 -> 37.6 mm
Changed lines of the file:
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@@
   (segment (start 111 71.93125) (end 111 71.9) (width 0.762) (layer "B.Cu") (net 5))
   (segment (start 111 71.9) (end 98.7 59.6) (width 0.762) (layer "B.Cu") (net 5))
+  (segment (start 85.05 61.45) (end 85.05 73.05) (width 0.254) (layer "F.Cu") (net 6))
+  (segment (start 94.8 73.6) (end 93.4625 74.9375) (width 0.762) (layer "F.Cu") (net 6))
+  (segment (start 85.05 61.45) (end 79.7 56.1) (width 0.254) (layer "F.Cu") (net 6))
+  (segment (start 93.4625 74.9375) (end 92 74.9375) (width 0.762) (layer "F.Cu") (net 6))
+  (segment (start 79.7 56.1) (end 79.7 53.735) (width 0.254) (layer "F.Cu") (net 6))
+  (segment (start 86.9375 74.9375) (end 88.8 74.9375) (width 0.254) (layer "F.Cu") (net 6))
+  (segment (start 96.4 73.6) (end 94.8 73.6) (width 0.762) (layer "F.Cu") (net 6))
+  (segment (start 88.4625 61.45) (end 85.05 61.45) (width 0.254) (layer "F.Cu") (net 6))
+  (segment (start 88.8 74.9375) (end 92 74.9375) (width 0.762) (layer "F.Cu") (net 6))
+  (segment (start 85.05 73.05) (end 86.9375 74.9375) (width 0.254) (layer "F.Cu") (net 6))
   (segment (start 88.8 69.5375) (end 88.8 73.0625) (width 0.508) (layer "F.Cu") (net 7))
   (segment (start 92 69.5375) (end 92 73.0625) (width 0.508) (layer "F.Cu") (net 8))
@@
   (segment (start 174.355999 146.818999) (end 185.293499 146.818999) (width 0.508) (layer "F.Cu") (net 85))
   (segment (start 226.148999 95.051001) (end 225 96.2) (width 0.762) (layer "F.Cu") (net 86))
-  (segment (start 219.209999 97.721499) (end 219.278501 97.721499) (width 0.762) (layer "F.Cu") (net 86))
   (segment (start 226.148999 93.750999) (end 226.148999 95.051001) (width 0.762) (layer "F.Cu") (net 86))
   (segment (start 225 96.2) (end 220.731498 96.2) (width 0.762) (layer "F.Cu") (net 86))
@@
   )
   (zone (net 1) (net_name "+3V3") (layer "F.Cu") (hatch edge 0.508)
-    (priority 1)
-    (connect_pads yes (clearance 0.3))
+    (priority 2)
+    (connect_pads yes (clearance 0.6))
     (min_thickness 0.254) (filled_areas_thickness no)
-    (fill yes (thermal_gap 0.508) (thermal_bridge_width 0.508))
+    (fill yes (thermal_gap 0.508) (thermal_bridge_width 0.508) (smoothing chamfer) (radius 0.25))
     (polygon
       (pts
@@
         (xy 114.4 62.8)
         (xy 111.5 62.8)
-        (xy 111.5 61.1)
-        (xy 115.7 56.8)
-        (xy 122.1 56.8)
+        (xy 111.5 60.8)
+        (xy 115.7 56.5)
+        (xy 122.1 56.5)
       )
     )
@@
       )
     )
+  )
+  (zone (net 2) (net_name "GND") (layer "F.Cu") (hatch edge 0.508)
+    (priority 1)
+    (connect_pads yes (clearance 0.4))
+    (min_thickness 0.254) (filled_areas_thickness no)
+    (fill yes (thermal_gap 0.508) (thermal_bridge_width 0.508) (smoothing chamfer) (radius 0.25))
+    (polygon
+      (pts
+        (xy 130.984491 61.412529)
+        (xy 123.404374 61.408671)
+        (xy 122.3 60.3)
+        (xy 122.3 55.7)
+        (xy 106.1 55.7)
+        (xy 106.1 51.9)
+        (xy 116.9 51.9)
+        (xy 116.9 48.3)
+        (xy 130.88302 48.306325)
+      )
+    )

Commit message: final
Parts:
- moved R28 1.80 mm to (92.7, 79.2)
- moved R8 1.21 mm to (226.4, 75.0)
Routing:
- net +3V3: track 63.3 -> 741.2 mm, vias 3 -> 16
- net +5V: track 45.6 -> 293.7 mm, vias 0 -> 6
- net RXD0: track 0.00 -> 71.7 mm, vias 0 -> 2
- net TXD0: track 0.00 -> 61.7 mm, vias 0 -> 2
- net IO27: track 15.0 -> 65.3 mm, vias 0 -> 1
- net IO0: track 0.00 -> 44.3 mm, vias 0 -> 2
- net EN: track 29.2 -> 66.5 mm, vias 0 -> 2
- net D+: track 0.00 -> 30.6 mm
- net D-: track 0.00 -> 30.6 mm
- net DTR: track 2.17 -> 29.7 mm, vias 0 -> 2
- net RTS: track 2.17 -> 20.5 mm
- net Net-(R4-Pad1): track 0.00 -> 13.7 mm, vias 0 -> 2
- net GND: track 63.4 -> 72.5 mm, vias 40 -> 69
- net VBUS: track 37.6 -> 43.7 mm, vias 0 -> 2
- net Net-(Q7-Pad3): track 19.4 -> 22.0 mm
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- added copper zone on F.Cu, net VBUS
