File: KiCad files/ESP32IoTPlatform.kicad_pcb (KiCad board)
At the start: 2 copper layers, 190 x 105.2 mm, 126 parts, among them IC1 ME6211C33M5G, J1 USB_B_Micro, J10 Conn_01x11_Female, J11 Conn_01x11_Male, J12 Conn_01x11_Male, J2 Screw_Terminal_01x03, J3 Screw_Terminal_01x02, J4 Screw_Terminal_01x02, J5 Conn_01x04_Female, J6 OLED, J7 Conn_01x05_Female, J8 Conn_01x05_Male, J9 Conn_01x11_Female, K1 SANYOU_SRD_Form_C, Q1 CJ2301, Q2 S8050G, Q3 IRLZ44N, Q4 SI2302DS, Q5 SI2302DS, Q6 Q_DUAL_NPN_UMH3N, Q7 Q_DUAL_PNP_BCM857BS, Q8 CJ2301, SW1 SW_Push, SW10 SW_x02, SW11 SW_x03, SW14 SW_x01, SW15 SW_x01, SW16 SW_x01, SW17 SW_x05, SW18 SW_x01, SW19 SW_x04, SW2 SW_x02, SW3 SW_x02, SW4 SW_x02, SW5 SW_x01, SW6 SW_x01, SW7 SW_x01, SW8 SW_x01, SW9 SW_x02, T1 SKRHABE010, U1 ESP32-WROOM-32D, U2 CP2104, U3 TP4054, U4 BME280, U5 MPU-6050, U6 PC817, U7 L80-M39

Commit message: done
Routing:
- net +3V3: track 741.2 -> 789.7 mm
- net +5V: track 293.7 -> 275.4 mm
- net VBUS: track 43.7 -> 39.6 mm
- net IO22: track 180.7 -> 179.0 mm
- net IO26: track 73.0 -> 71.8 mm
- net DTR: track 29.7 -> 29.1 mm
- net IO21: track 177.4 -> 176.9 mm

Commit message: v4.0
Parts:
- H1, H2, H3, H4: footprint MountingHole:MountingHole_3.2mm_M3_Pad_Via -> ESP32IoTPlatform:MountingHole_3.2mm_M3_Pad_Via_edited
Routing:
- net IO25: track 122.4 -> 116.8 mm
- net IO15: track 81.4 -> 84.8 mm
- net IO22: track 179.0 -> 179.8 mm
