File: KiCad files/ESP32IoTPlatform.kicad_sch (KiCad schematic)
At the start: 62 parts, among them IC1 ME6211C33M5G, J1 USB_B_Micro, J2 Screw_Terminal_01x03, K1 SANYOU_SRD_Form_C, Q1 CJ2301, Q2 S8050G, SW1 SW_Push, SW2 SW_x02, SW3 SW_x02, SW4 SW_x02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

Commit message: Update
Parts:
- removed C1, C12, C15, C16, C17, C18, C4, C8, C9: 100n/50V, Capacitor_SMD:C_0805_2012Metric, symbol Device:C_Small
- removed C10: 10n/6.3V, Capacitor_SMD:C_0805_2012Metric, symbol Device:C_Small
- removed C11: 2200p/50V, Capacitor_SMD:C_0805_2012Metric, symbol Device:C_Small
- removed C13, C14, C2: 1u/50V, Capacitor_SMD:C_0805_2012Metric, symbol Device:C_Small
- removed C3: 1000u, Capacitor_Tantalum_SMD:CP_EIA-7343-31_Kemet-D, symbol Device:CP_Small
- removed C5, C6, C7: 10u/16V, Capacitor_SMD:C_0805_2012Metric, symbol Device:C_Small
- removed D1: Green, LED_SMD:LED_0805_2012Metric, symbol Device:LED_Small
- removed D10, D2: Red, LED_SMD:LED_0805_2012Metric, symbol Device:LED_Small
- removed D11: S1BB-13-F, Diode_SMD:D_SMA, symbol Device:D_Small
- removed D3: Orange, LED_SMD:LED_0805_2012Metric, symbol Device:LED_Small
- removed D4: B5819WS, Diode_SMD:D_SOD-323, symbol Diode:1N5819
- removed D5, D6, D7, D8: WS2812B, LED_SMD:LED_WS2812B_PLCC4_5.0x5.0mm_P3.2mm, symbol LED:WS2812B
- removed D9: Blue, LED_SMD:LED_1206_3216Metric, symbol Device:LED_Small
- removed IC1: ME6211C33M5G, Package_TO_SOT_SMD:SOT-23-5, symbol ESP32IoTPlatform_simboli:ME6211C33M5G
- removed J1: USB_B_Micro, ESP32IoTPlatform:USB_Micro-AB_Molex_47590-0001, symbol Connector:USB_B_Micro
- removed J2: Screw_Terminal_01x03, TerminalBlock_Phoenix:TerminalBlock_Phoenix_MKDS-1,5-3-5.08_1x03_P5.08mm_Horizontal, symbol Connector:Screw_Terminal_01x03
- removed JST1: JST2.0, Connector_JST:JST_PH_B2B-PH-K_1x02_P2.00mm_Vertical, symbol Connector_Generic:Conn_01x02
- removed K1: SANYOU_SRD_Form_C, ESP32IoTPlatform:Relay_SPDT_SANYOU_SRD_Series_Form_C, symbol Relay:SANYOU_SRD_Form_C
- removed Q1: CJ2301, Package_TO_SOT_SMD:SOT-23, symbol Transistor_FET:Si2319CDS
- removed Q2: S8050G, Package_TO_SOT_SMD:SOT-23, symbol Transistor_BJT:S8050
- removed R1, R10, R6, R7, R8, R9: 10k, Resistor_SMD:R_0805_2012Metric, symbol Device:R_Small
- removed R11: 80R, Resistor_SMD:R_0805_2012Metric, symbol Device:R_Small
- removed R12, R13: 1k, Resistor_SMD:R_0805_2012Metric, symbol Device:R_Small
- removed R2, R3: 330R, Resistor_SMD:R_0805_2012Metric, symbol Device:R_Small
- removed R4: 243R, Resistor_SMD:R_0805_2012Metric, symbol Device:R_Small
- removed R5: 2k, Resistor_SMD:R_0805_2012Metric, symbol Device:R_Small
- removed SW1: SW_Push, Button_Switch_SMD:SW_SPST_PTS645, symbol Switch:SW_Push
- removed SW2, SW3, SW4: SW_x02, Button_Switch_SMD:SW_DIP_SPSTx02_Slide_6.7x6.64mm_W6.73mm_P2.54mm_LowProfile_JPin, symbol Switch:SW_DIP_x02
- removed SW5, SW6, SW7: SW_x01, Button_Switch_SMD:SW_DIP_SPSTx01_Slide_6.7x4.1mm_W6.73mm_P2.54mm_LowProfile_JPin, symbol Switch:SW_DIP_x01
- removed U1: ESP32-WROOM-32D, RF_Module:ESP32-WROOM-32, symbol RF_Module:ESP32-WROOM-32D
- removed U2: CP2104, Package_DFN_QFN:QFN-24-1EP_4x4mm_P0.5mm_EP2.6x2.6mm, symbol Interface_USB:CP2104
- removed U3: TP4054, Package_TO_SOT_SMD:TSOT-23-5, symbol Battery_Management:LTC4054ES5-4.2
- removed U4: BME280, ESP32IoTPlatform:Bosch_LGA-8_2.5x2.5mm_P0.65mm_ClockwisePinNumbering, symbol Sensor:BME280
- removed U5: MPU-6050, Sensor_Motion:InvenSense_QFN-24_4x4mm_P0.5mm, symbol Sensor_Motion:MPU-6050
- removed U6: PC817, Package_DIP:DIP-4_W7.62mm, symbol Isolator:PC817
- added H1, H2, H3, H4: MountingHole, MountingHole:MountingHole_3.2mm_M3_Pad_Via, symbol Mechanical:MountingHole
Connections:
- no-connect marks 23 -> 0
Other:
- removed sheet Sheet2
- added sheet Aktuatori (aktuatori.kicad_sch)
- added sheet I2C (I2C.kicad_sch)
- added sheet LEDs (LEDs.kicad_sch)
- added sheet Napajanje (napajanje.kicad_sch)
- added sheet SPI (SPI.kicad_sch)
- added sheet Senzori (senzori.kicad_sch)
- added sheet mcu (mcu.kicad_sch)
- added sheet usb-uart (usb-uart.kicad_sch)
- note added: "Aktuatori"
- note added: "I2C uređaji"
- note added: "LED"
- note added: "Napajanje"
- note added: "RUPE"
- note added: "SPI uređaji"
- note added: "Senzori"
- note added: "uC"
- note removed: "3.3V REGULATOR NAPONA"
- note removed: "BME280"
- note removed: "ESP32"
- note removed: "I2C PRITEZNI OTPORNICI"
- note removed: "MPU-6050"
- note removed: "Note: VDD"
- note removed: "PUNJAČ BATERIJE"
- note removed: "RELEJ"
- note removed: "SVJETLEĆA DIODA"
- note removed: "Sheet 2"
- note removed: "VIŠEBOJNE SVJETLEĆE DIODE"
- note removed: "microUSB"
- company: (none) -> TVZ
- title: (none) -> ESP32IoTPlatform

Commit message: done
Other:
- note added: "ESP32IoTPlatform V4.0"
Changed lines of the file:
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@@
     (effects (font (size 5 5) (thickness 1) bold) (justify right bottom))
+  )
+  (text "ESP32IoTPlatform V4.0" (at 233.045 31.75 180)
+    (effects (font (size 10 10) (thickness 1) bold) (justify right bottom))
   )
   (text "I2C uređaji" (at 167.64 67.31 180)

Commit message: v4.0
Parts:
- H1, H2, H3, H4: footprint MountingHole:MountingHole_3.2mm_M3_Pad_Via -> ESP32IoTPlatform:MountingHole_3.2mm_M3_Pad_Via_edited
Changed lines of the file:
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@@
       (effects (font (size 1.27 1.27)) (justify left))
     )
-    (property "Footprint" "MountingHole:MountingHole_3.2mm_M3_Pad_Via" (id 2) (at 260.985 159.385 0)
+    (property "Footprint" "ESP32IoTPlatform:MountingHole_3.2mm_M3_Pad_Via_edited" (id 2) (at 260.985 159.385 0)
       (effects (font (size 1.27 1.27)) hide)
     )
@@
       (effects (font (size 1.27 1.27)) (justify left))
     )
-    (property "Footprint" "MountingHole:MountingHole_3.2mm_M3_Pad_Via" (id 2) (at 260.985 144.145 0)
+    (property "Footprint" "ESP32IoTPlatform:MountingHole_3.2mm_M3_Pad_Via_edited" (id 2) (at 260.985 144.145 0)
       (effects (font (size 1.27 1.27)) hide)
     )
@@
       (effects (font (size 1.27 1.27)) (justify left))
     )
-    (property "Footprint" "MountingHole:MountingHole_3.2mm_M3_Pad_Via" (id 2) (at 260.985 149.225 0)
+    (property "Footprint" "ESP32IoTPlatform:MountingHole_3.2mm_M3_Pad_Via_edited" (id 2) (at 260.985 149.225 0)
       (effects (font (size 1.27 1.27)) hide)
     )
@@
       (effects (font (size 1.27 1.27)) (justify left))
     )
-    (property "Footprint" "MountingHole:MountingHole_3.2mm_M3_Pad_Via" (id 2) (at 260.985 154.305 0)
+    (property "Footprint" "ESP32IoTPlatform:MountingHole_3.2mm_M3_Pad_Via_edited" (id 2) (at 260.985 154.305 0)
       (effects (font (size 1.27 1.27)) hide)
     )
@@
     )
     (path "/87c6b209-8d32-4b59-b036-8912faa222a7"
-      (reference "H1") (unit 1) (value "MountingHole") (footprint "MountingHole:MountingHole_3.2mm_M3_Pad_Via")
+      (reference "H1") (unit 1) (value "MountingHole") (footprint "ESP32IoTPlatform:MountingHole_3.2mm_M3_Pad_Via_edited")
     )
     (path "/bb106a84-610d-45d8-905c-d888aa48e835"
-      (reference "H2") (unit 1) (value "MountingHole") (footprint "MountingHole:MountingHole_3.2mm_M3_Pad_Via")
+      (reference "H2") (unit 1) (value "MountingHole") (footprint "ESP32IoTPlatform:MountingHole_3.2mm_M3_Pad_Via_edited")
     )
     (path "/ecfcee40-6e37-4b9a-823d-5249874fbcab"
-      (reference "H3") (unit 1) (value "MountingHole") (footprint "MountingHole:MountingHole_3.2mm_M3_Pad_Via")
+      (reference "H3") (unit 1) (value "MountingHole") (footprint "ESP32IoTPlatform:MountingHole_3.2mm_M3_Pad_Via_edited")
     )
     (path "/77643c0d-528b-4bab-8e3f-c42edaed28d7"
-      (reference "H4") (unit 1) (value "MountingHole") (footprint "MountingHole:MountingHole_3.2mm_M3_Pad_Via")
+      (reference "H4") (unit 1) (value "MountingHole") (footprint "ESP32IoTPlatform:MountingHole_3.2mm_M3_Pad_Via_edited")
     )
     (path "/5bcf160e-42fa-48f0-b959-5331edc20809/e69f0cef-fdd0-45f7-9147-2d21654f92e6"
